File: 3x3 midi mixer fader.kicad_sch (KiCad schematic)
At the start: 76 parts, among them J1 B1, J2 B2, J3 B3, J4 B4, Q0 BSS138, U0 ADS1115IDGS, U1 W25Q128JVS

Commit message: Add files via upload
Parts:
- removed A0: RaspberryPi_Pico, Module:RaspberryPi_Pico_Common_SMD, symbol MCU_Module:RaspberryPi_Pico
- removed C14, C16, C17, C19, C20: 0.1uF, Capacitor_SMD:C_0603_1608Metric_Pad1.08x0.95mm_HandSolder, symbol Device:C
- removed C2: 10uF, Capacitor_THT:CP_Radial_D5.0mm_P2.50mm, symbol Device:C
- removed Q0: BSS138, Package_TO_SOT_SMD:SOT-23, symbol Transistor_FET:BSS138
- removed R8: 4.7k, Resistor_SMD:R_0603_1608Metric_Pad0.98x0.95mm_HandSolder, symbol Device:R
- removed RGB0: WS2812B, PCM_marbastlib-mx:LED_MX_6028R-ROT, symbol PCM_marbastlib-mx:MX_SK6812MINI-E
- removed U0: ADS1115IDGS, Package_SO:TSSOP-10_3x3mm_P0.5mm, symbol Analog_ADC:ADS1115IDGS
- added 1V1: 1.1V, TestPoint:TestPoint_Pad_1.5x1.5mm, symbol Connector:TestPoint
- added 3V3: 3.3V, TestPoint:TestPoint_Pad_1.5x1.5mm, symbol Connector:TestPoint
- added 5V1: 5V, TestPoint:TestPoint_Pad_1.5x1.5mm, symbol Connector:TestPoint
- added C21, C25: 100n, Capacitor_SMD:C_0402_1005Metric, symbol Device:C
- added C26: 15p, Capacitor_SMD:C_0402_1005Metric, symbol Device:C
- added C6: 100n, Capacitor_SMD:C_0603_1608Metric, symbol Device:C
- added GND1: GND, TestPoint:TestPoint_Pad_1.5x1.5mm, symbol Connector:TestPoint
- added J1: USB_C_Receptacle_USB2.0_16P, Connector_USB:USB_C_Receptacle_HRO_TYPE-C-31-M-12, symbol Connector:USB_C_Receptacle_USB2.0_16P
- added J6: Conn_01x04, Connector_JST:JST_XH_B4B-XH-A_1x04_P2.50mm_Vertical, symbol Connector_Generic:Conn_01x04
- added J7: Conn_01x04, Connector_PinHeader_2.54mm:PinHeader_1x04_P2.54mm_Vertical, symbol Connector_Generic:Conn_01x04
- added R15, R18: 27, Resistor_SMD:R_0603_1608Metric, symbol Device:R
- added R17: 3.3k, Resistor_SMD:R_0603_1608Metric, symbol Device:R
- added R21: 1k, Resistor_SMD:R_0402_1005Metric, symbol Device:R
- added R23: 10k, Resistor_SMD:R_0603_1608Metric, symbol Device:R
- added R6: 5.1K, Resistor_SMD:R_0603_1608Metric, symbol Device:R
- added RGB5: WS2812B, PCM_marbastlib-mx:LED_MX_6028R-ROT, symbol PCM_marbastlib-mx:MX_SK6812MINI-E
- added SW1, SW2: SW_SPST, Button_Switch_SMD:SW_SPST_SKQG_WithStem, symbol Switch:SW_SPST
- added U1: USBLC6-2SC6, Package_TO_SOT_SMD:SOT-23-6, symbol Power_Protection:USBLC6-2SC6
- added U2: W25Q16JVSS, Package_SO:SOIC-8_5.3x5.3mm_P1.27mm, symbol Memory_Flash:W25Q16JVSS
- added U4: XC6206PxxxMR, Package_TO_SOT_SMD:SOT-23-3, symbol Regulator_Linear:XC6206PxxxMR
- added U6: RP2040, Package_DFN_QFN:QFN-56-1EP_7x7mm_P0.4mm_EP3.2x3.2mm_ThermalVias, symbol MCU_RaspberryPi:RP2040
- added Y1: Crystal_GND24, Crystal:Crystal_SMD_3225-4Pin_3.2x2.5mm, symbol Device:Crystal_GND24
- C1: renamed from C3; value 10uF -> 100n; footprint Capacitor_THT:CP_Radial_D5.0mm_P2.50mm -> Capacitor_SMD:C_0603_1608Metric; KiLib_Generator (none) -> capacitor/THT/other
- C10, C11, C12, C18, C22, C24, C9: value 0.1uF -> 100n; footprint Capacitor_SMD:C_0603_1608Metric_Pad1.08x0.95mm_HandSolder -> Capacitor_SMD:C_0402_1005Metric; KiLib_Generator (none) -> SMD_2terminal_chip_molded
- C13, C15: value 0.1uF -> 1u; footprint Capacitor_SMD:C_0603_1608Metric_Pad1.08x0.95mm_HandSolder -> Capacitor_SMD:C_0402_1005Metric; KiLib_Generator (none) -> SMD_2terminal_chip_molded
- C2: renamed from C8; value 10uF -> 100n; footprint Capacitor_THT:CP_Radial_D5.0mm_P2.50mm -> Capacitor_SMD:C_0603_1608Metric; KiLib_Generator (none) -> capacitor/THT/other
- C23: value 0.1uF -> 15p; footprint Capacitor_SMD:C_0603_1608Metric_Pad1.08x0.95mm_HandSolder -> Capacitor_SMD:C_0402_1005Metric; KiLib_Generator (none) -> SMD_2terminal_chip_molded
- C3: renamed from C6; value 10uF -> 100n; footprint Capacitor_THT:CP_Radial_D5.0mm_P2.50mm -> Capacitor_SMD:C_0603_1608Metric; KiLib_Generator (none) -> capacitor/THT/other
- C4: value 0.1uF -> 100n; footprint Capacitor_SMD:C_0603_1608Metric_Pad1.08x0.95mm_HandSolder -> Capacitor_SMD:C_0603_1608Metric; KiLib_Generator (none) -> capacitor/THT/other
- C5, C7: value 0.1uF -> 10u; footprint Capacitor_SMD:C_0603_1608Metric_Pad1.08x0.95mm_HandSolder -> Capacitor_SMD:C_0603_1608Metric; KiLib_Generator (none) -> SMD_2terminal_chip_molded
- C8: renamed from C21; value 0.1uF -> 100n; footprint Capacitor_SMD:C_0603_1608Metric_Pad1.08x0.95mm_HandSolder -> Capacitor_SMD:C_0603_1608Metric; KiLib_Generator (none) -> SMD_2terminal_chip_molded
- J2: renamed from J1; footprint Connector_JST:JST_ZH_B3B-ZR_1x03_P1.50mm_Vertical -> Connector_JST:JST_XH_B3B-XH-A_1x03_P2.50mm_Vertical; KiLib_Generator (none) -> connector/JST
- J3: footprint Connector_JST:JST_ZH_B3B-ZR_1x03_P1.50mm_Vertical -> Connector_JST:JST_XH_B3B-XH-A_1x03_P2.50mm_Vertical; KiLib_Generator (none) -> connector/JST
- J4: renamed from J2; footprint Connector_JST:JST_ZH_B3B-ZR_1x03_P1.50mm_Vertical -> Connector_JST:JST_XH_B3B-XH-A_1x03_P2.50mm_Vertical; KiLib_Generator (none) -> connector/JST
- J5: renamed from J4; footprint Connector_JST:JST_ZH_B3B-ZR_1x03_P1.50mm_Vertical -> Connector_JST:JST_XH_B3B-XH-A_1x03_P2.50mm_Vertical; KiLib_Generator (none) -> connector/JST
- R10: value 10k -> 1K; footprint Resistor_SMD:R_0603_1608Metric_Pad0.98x0.95mm_HandSolder -> Resistor_SMD:R_0603_1608Metric; KiLib_Generator (none) -> SMD_2terminal_chip_molded
- R11: value 220 -> DNP; footprint Resistor_SMD:R_0603_1608Metric_Pad0.98x0.95mm_HandSolder -> Resistor_SMD:R_0603_1608Metric; KiLib_Generator (none) -> SMD_2terminal_chip_molded
- R12: renamed from R15; footprint Resistor_SMD:R_0603_1608Metric_Pad0.98x0.95mm_HandSolder -> Resistor_SMD:R_0603_1608Metric; KiLib_Generator (none) -> SMD_2terminal_chip_molded
- R13: renamed from R5; footprint Resistor_SMD:R_0603_1608Metric_Pad0.98x0.95mm_HandSolder -> Resistor_SMD:R_0603_1608Metric; KiLib_Generator (none) -> SMD_2terminal_chip_molded
- R14: value 10k -> 3.3k; footprint Resistor_SMD:R_0603_1608Metric_Pad0.98x0.95mm_HandSolder -> Resistor_SMD:R_0603_1608Metric
- R16: footprint Resistor_SMD:R_0603_1608Metric_Pad0.98x0.95mm_HandSolder -> Resistor_SMD:R_0603_1608Metric; KiLib_Generator (none) -> SMD_2terminal_chip_molded
- R19: renamed from R12; footprint Resistor_SMD:R_0603_1608Metric_Pad0.98x0.95mm_HandSolder -> Resistor_SMD:R_0603_1608Metric; KiLib_Generator (none) -> SMD_2terminal_chip_molded
- R20: renamed from R17; footprint Resistor_SMD:R_0603_1608Metric_Pad0.98x0.95mm_HandSolder -> Resistor_SMD:R_0603_1608Metric; KiLib_Generator (none) -> SMD_2terminal_chip_molded
- R22: renamed from R6; footprint Resistor_SMD:R_0603_1608Metric_Pad0.98x0.95mm_HandSolder -> Resistor_SMD:R_0603_1608Metric; KiLib_Generator (none) -> SMD_2terminal_chip_molded
- R24: renamed from R18; footprint Resistor_SMD:R_0603_1608Metric_Pad0.98x0.95mm_HandSolder -> Resistor_SMD:R_0603_1608Metric; KiLib_Generator (none) -> SMD_2terminal_chip_molded
- R25: renamed from R13; footprint Resistor_SMD:R_0603_1608Metric_Pad0.98x0.95mm_HandSolder -> Resistor_SMD:R_0603_1608Metric; KiLib_Generator (none) -> SMD_2terminal_chip_molded
- R7: value 4.7k -> 5.1K; footprint Resistor_SMD:R_0603_1608Metric_Pad0.98x0.95mm_HandSolder -> Resistor_SMD:R_0603_1608Metric; KiLib_Generator (none) -> SMD_2terminal_chip_molded
- R9: footprint Resistor_SMD:R_0603_1608Metric_Pad0.98x0.95mm_HandSolder -> Resistor_SMD:R_0603_1608Metric
- RGB1: footprint PCM_marbastlib-mx:LED_MX_6028R-ROT -> PCM_marbastlib-mx:LED_MX_6028R
- RGB2: renamed from RGB3; footprint PCM_marbastlib-mx:LED_MX_6028R-ROT -> PCM_marbastlib-mx:LED_MX_6028R
- RGB3: renamed from RGB5; footprint PCM_marbastlib-mx:LED_MX_6028R-ROT -> PCM_marbastlib-mx:LED_MX_6028R
- RGB7: renamed from RGB4; footprint PCM_marbastlib-mx:LED_MX_6028R-ROT -> PCM_marbastlib-mx:LED_MX_6028R
- RGB8: renamed from RGB7; footprint PCM_marbastlib-mx:LED_MX_6028R-ROT -> PCM_marbastlib-mx:LED_MX_6028R
- RGB9: renamed from RGB8; footprint PCM_marbastlib-mx:LED_MX_6028R-ROT -> PCM_marbastlib-mx:LED_MX_6028R
- U3: renamed from U1; value W25Q128JVS -> 24LC256; symbol Memory_Flash:W25Q128JVS -> Memory_EEPROM:24LC256; KiLib_Generator (none) -> package/gullwing
- renumbered D5 to D1, D1 to D2, D0 to D3, D8 to D4, D7 to D5, D3 to D6, D2 to D7, D4 to D8, D6 to D9, R4 to R3, R3 to R4, RGB2 to RGB4, S8 to S1, S1 to S2, S0 to S3, S7 to S4, S3 to S6, S2 to S7, S6 to S8, S4 to S9
Connections:
- net SCL is gone; now on net GND: R7.2
- net SPI_MISO is gone; now on net GND: U3.2 (A1)
- net SPI_MOSI is gone; now on net EEPROM_SDA: U3.5 (SDA)
- net WS2812IN_LV is gone; now on net ~{QSPI_SS}: R10.2
- net +3.3V: now also C11.1, C12.1, C15.1, C18.1, C22.1, C24.1, R11.1, R13.2, R19.2, R22.2, 3V3.1, C21.1, C6.1, J7.4 (Pin_4), R17.1, R23.1, U2.8 (VCC), U4.2 (VO), U6.1 (IOVDD), U6.10 (IOVDD), U6.22 (IOVDD), U6.33 (IOVDD), U6.42 (IOVDD), U6.43 (ADC_AVDD), U6.44 (VREG_VIN), U6.48 (USB_VDD), U6.49 (IOVDD); no longer C13.1, C5.1, R10.1, R13.1, R19.1, R22.1, R7.1, U3.3 (~{WP}/IO_{2}), U3.7 (~{HOLD}/~{RESET}/IO_{3})
- net +5V: now also C5.1, 5V1.1, J1.A4 (VBUS), J1.A9 (VBUS), J1.B4 (VBUS), J1.B9 (VBUS), J6.1 (Pin_1), RGB5.1 (VDD), U1.5 (VBUS), U4.3 (VI); no longer C10.1, C11.1, C12.1, C18.1, C22.1, C23.1, C24.1, R9.1
- net GND: now also R9.2, U3.1 (A0), U3.3 (A2), C21.2, C25.2, C26.2, C6.2, GND1.1, J1.A1 (GND), J1.A12 (GND), J1.B1 (GND), J1.B12 (GND), J1.SH (SHIELD), J6.4 (Pin_4), J7.1 (Pin_1), R6.2, RGB5.4 (VSS), SW1.1 (A), SW2.1 (A), U1.2 (GND), U2.4 (GND), U4.1 (GND), U6.19 (TESTEN), U6.57 (GND), Y1.2 (G), Y1.4 (G)
- net at RGB6.2 (DOUT): now also RGB5.3 (DIN)
- net WS2812_RGB: now reaches RGB1.3 (DIN)
- net WS2812_RGB: now also U6.30 (GPIO19); no longer R11.1
- net at RGB4.3 (DIN): now also RGB5.2 (DOUT)
- net B1 renamed Button_1
- net Button_1: now also R13.1, U6.8 (GPIO6); no longer R13.2
- net B2 renamed Button_2
- net Button_2: now also R22.1, U6.9 (GPIO7); no longer R22.2
- net B3 renamed Button_3
- net Button_3: now also R19.1, U6.11 (GPIO8); no longer R19.2
- net B4 renamed Button_4
- net Button_4: now also U6.12 (GPIO9)
- net Column 1 renamed Col_1
- net Col_1: now also U6.35 (GPIO23)
- net Column 2 renamed Col_2
- net Col_2: now also U6.36 (GPIO24)
- net Column 3 renamed Col_3
- net Col_3: now also U6.37 (GPIO25)
- net Fader 1 renamed Fader_1
- net Fader_1: now also U6.38 (GPIO26/ADC0); no longer C15.1
- net Fader 2 renamed Fader_2
- net Fader_2: now also U6.39 (GPIO27/ADC1)
- net Fader 3 renamed Fader_3
- net Fader_3: now also U6.40 (GPIO28/ADC2)
- net Fader 4 renamed Fader_4
- net Fader_4: now also U6.41 (GPIO29/ADC3)
- net LED1 renamed LED_1
- net LED_1: now also U6.13 (GPIO10)
- net LED2 renamed LED_3
- net LED_3: now also U6.15 (GPIO12)
- net LED3 renamed LED_2
- net LED_2: now also U6.14 (GPIO11)
- net LED4 renamed LED_4
- net LED_4: now also U6.16 (GPIO13)
- net Row 1 renamed Row_1
- net Row_1: now also U6.34 (GPIO22)
- net Row 2 renamed Row_2
- net Row_2: now also U6.32 (GPIO21)
- net Row 3 renamed Row_3
- net Row_3: now also U6.31 (GPIO20)
- net SPI_CLK renamed EEPROM_SCL
- net EEPROM_SCL: now also J7.2 (Pin_2), R17.2, U6.3 (GPIO1)
- net SPI_CS renamed EEPROM_SDA
- net EEPROM_SDA: now also J7.3 (Pin_3), U6.2 (GPIO0); no longer U3.1 (~{CS})
- net WS2812IN_HV renamed ~{QSPI_SS}
- net ~{QSPI_SS}: now also U2.1 (~{CS}), U6.56 (~{QSPI_SS}); no longer R9.2
- new net: R9.1, U3.7 (WP)
- new net: C26.1, U6.20 (XIN), Y1.1
- new net: R21.2, U6.21 (XOUT)
- new net: R18.1, U6.46 (USB_DM)
- new net: R15.2, U6.47 (USB_DP)
- new net: C23.1, R21.1, Y1.3
- new net: R10.1, SW1.2 (B)
- new net: J1.A5 (CC1), R7.1
- new net: J1.B5 (CC2), R6.1
- new net +1V1: 1V1.1, C10.1, C13.1, C25.1, U6.23 (DVDD), U6.45 (VREG_VOUT), U6.50 (DVDD)
- new net QSPI_SCLK: U2.6 (CLK), U6.52 (QSPI_SCLK)
- new net QSPI_SD1: U2.2 (DO/IO_{1}), U6.55 (QSPI_SD1)
- new net QSPI_SD2: U2.3 (~{WP}/IO_{2}), U6.54 (QSPI_SD2)
- new net QSPI_SD3: U2.7 (~{HOLD}/~{RESET}/IO_{3}), U6.51 (QSPI_SD3)
- new net QSPI_SDO: U2.5 (DI/IO_{0}), U6.53 (QSPI_SD0)
- new net SWCLK: U6.24 (SWCLK)
- new net SWDIO: U6.25 (SWDIO)
- new net USB_CON_D+: J1.A6 (D+), J1.B6 (D+), J6.3 (Pin_3), U1.3 (I/O2)
- new net USB_CON_D-: J1.A7 (D-), J1.B7 (D-), J6.2 (Pin_2), U1.1 (I/O1)
- new net USB_D+: R15.1, U1.4 (I/O2)
- new net USB_D-: R18.2, U1.6 (I/O1)
- new net ~{RESET}: R23.2, SW2.2 (B), U6.26 (RUN)
- no-connect marks 0 -> 14
Other:
- note added: "Make sure C13 is close to pin 45"
- note added: "Make sure C15 is close to pin 44"
- note added: "R11 is uneccessary for this EEPROM"
- note added: "RP2040 FLASH"
- note added: "USB"
- note added: "Ws2812B"
- note removed: "ADC"
- note removed: "Level Shifter"
- moved on the sheet: C1, C2, C3, C8, D1, D2, D3, D4, D5, D6, D7, D8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
